Commit message: 08/12

File: cva_gym/description/turtlebot3/urdf/turtlebot3_waffle_pi.urdf.xacro (robot description, xacro)
@@ -7,5 +7,5 @@
       <origin xyz="-0.064 0 0.055" rpy="0 0 0"/>
         <geometry>
-          <box size="0.33 0.28 0.100"/>
+          <box size="0.33 0.28 0.010"/>
         </geometry>
     </collision>
